File: board/board.kicad_pcb (KiCad board)
At the start: 2 copper layers, 21 x 13 mm, 1 part

Commit message: initial commit
Parts:
- added C1: 0.1uF, Capacitor_SMD:C_0603_1608Metric_Pad1.08x0.95mm_HandSolder, F.Cu at (142.2, 100.1)
- added J1: 011_GPIO, on_edge:on_edge_2x05_device, F.Cu at (161.0, 96.4)
- added Q1: SI2302DDS-T1-GE3, torque:FP-S-03946-MFG, F.Cu at (154.0, 97.7)
- added R1: 10k, Resistor_SMD:R_0603_1608Metric_Pad0.98x0.95mm_HandSolder, F.Cu at (145.1, 96.5)
- added R2: 10k, Resistor_SMD:R_0603_1608Metric_Pad0.98x0.95mm_HandSolder, F.Cu at (154.1, 95.0)
- added U1: SS443A, torque:FP-SS443A-MFG, F.Cu at (141.9, 96.5)
- moved LOGO1 0.90 mm to (149.1, 99.0)
Routing:
- net /SS443A/5V: track 0.00 -> 26.1 mm
- net Net-(R1-Pad2): track 0.00 -> 15.2 mm
- net /SS443A/OUT: track 0.00 -> 8.72 mm
- net GND: track 0.00 -> 8.03 mm, vias 0 -> 49
- net /SS443A/3V3: track 0.00 -> 4.84 mm, vias 0 -> 1
- added copper zone on B.Cu, net GND
- added copper zone on F.Cu, net GND
Other:
- outline, holes or cut-outs redrawn
- board text added: "b130_SS443A_hall_v01"
- board text added: "osf.011.gpio"
