File: board/board.kicad_pcb (KiCad board)
At the start: 2 copper layers, 21 x 13 mm, 7 parts, among them J1 011_GPIO, Q1 SI2302DDS-T1-GE3, U1 SS443A

Commit message: Update libraries
Parts:
- C1: value 0.1uF -> 100nF
Changed lines of the file:
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@@
   (net 8 "unconnected-(J1-Pad7)")
   (net 9 "/SS443A/3V3")
-  (net 10 "Net-(R1-Pad2)")
+  (net 10 "Net-(Q1-Pad1)")
   (footprint "on_edge:on_edge_2x05_device" (layer "F.Cu")
     (at 160.99943 96.435396 90)
@@
     (attr exclude_from_pos_files)
     (fp_text reference "J1" (at 0 1.2 90 unlocked) (layer "F.Fab")
-      (effects (font (size 0.7 0.7) (thickness 0.127)))
+      (effects (font (size 0.8 0.8) (thickness 0.127)))
     )
     (fp_text value "011_GPIO" (at 0 2 90 unlocked) (layer "F.Fab")
-      (effects (font (size 0.7 0.7) (thickness 0.127)))
+      (effects (font (size 0.8 0.8) (thickness 0.127)))
     )
     (fp_line (start -1 -4.05) (end -1 -3.323) (layer "F.SilkS") (width 0.153))
@@
         (gr_poly (pts
             (xy 0.5 -1.8)
+            (xy -0.5 -1.8)
             (xy 0.5 -1.9)
-            (xy -0.5 -1.8)
           ) (width 0) (fill yes))
       ))
@@
       (primitives
         (gr_poly (pts
+            (xy 0.5 -0.99)
+            (xy 0.48 -0.97)
+            (xy 0.44 -0.92)
+            (xy 0.4 -0.86)
+            (xy 0.37 -0.81)
+            (xy 0.35 -0.76)
+            (xy 0.33 -0.7)
+            (xy 0.31 -0.62)
             (xy 0.3 -0.51)
-            (xy 0.31 -0.62)
-            (xy 0.33 -0.7)
-            (xy 0.35 -0.76)
-            (xy 0.37 -0.81)
-            (xy 0.4 -0.86)
-            (xy 0.44 -0.92)
-            (xy 0.48 -0.97)
-            (xy 0.5 -0.99)
+            (xy 0.3 1.5)
+            (xy -0.5 1.5)
+            (xy -0.5 -2.3)
             (xy 0.5 -2.4)
-            (xy -0.5 -2.3)
-            (xy -0.5 1.5)
-            (xy 0.3 1.5)
           ) (width 0) (fill yes))
       ))
@@
       (primitives
         (gr_poly (pts
+            (xy 0.5 -1.8)
             (xy -0.5 -1.8)
             (xy -0.5 -1.9)
-            (xy 0.5 -1.8)
           ) (width 0) (fill yes))
       ))
@@
       (primitives
         (gr_poly (pts
+            (xy 0.5 -1.7)
             (xy -0.5 -1.7)
             (xy -0.5 -1.8)
-            (xy 0.5 -1.7)
           ) (width 0) (fill yes))
       ))
@@
       (connect_pads (clearance 0))
       (min_thickness 0.254)
-      (keepout (tracks allowed) (vias not_allowed) (pads allowed) (copperpour not_allowed) (footprints not_allowed))
+      (keepout (tracks allowed) (vias not_allowed) (pads allowed ) (copperpour not_allowed) (footprints not_allowed))
       (fill (thermal_gap 0.508) (thermal_bridge_width 0.508))
       (polygon
@@
     (property "Sheetname" "SS443A")
     (fp_text reference "Q1" (at 0 -3.3 90 unlocked) (layer "F.SilkS")
-      (effects (font (size 0.7 0.7) (thickness 0.127)) (justify left bottom))
+      (effects (font (size 0.8 0.8) (thickness 0.127)) (justify left bottom))
     )
     (fp_text value "SI2302DDS-T1-GE3" (at -1.3081 4.0005 180 unlocked) (layer "F.SilkS") hide
-      (effects (font (size 0.7 0.7) (thickness 0.127)) (justify left bottom))
+      (effects (font (size 0.8 0.8) (thickness 0.127)) (justify left bottom))
     )
     (fp_text user "${REFERENCE}" (at 0 0.139012 180 unlocked) (layer "User.5")
-      (effects (font (size 0.5 0.5) (thickness 0.1)) (justify left bottom))
+      (effects (font (size 0.8 0.8) (thickness 0.127)) (justify left bottom))
     )
     (fp_line (start -0.7 -0.298099) (end -0.7 0.298099) (layer "F.SilkS") (width 0.2))
@@
     (fp_line (start 1.45893 -1.62) (end -1.458928 -1.62) (layer "User.5") (width 0.2))
     (pad "1" smd rect (at -0.990628 -0.9525 180) (size 0.7366 0.5588) (layers "F.Cu" "F.Paste" "F.Mask")
-      (net 10 "Net-(R1-Pad2)") (pinfunction "G") (pintype "passive"))
+      (net 10 "Net-(Q1-Pad1)") (pinfunction "G") (pintype "passive"))
     (pad "2" smd rect (at -0.990628 0.9525 180) (size 0.7366 0.5588) (layers "F.Cu" "F.Paste" "F.Mask")
       (net 2 "GND") (pinfunction "S") (pintype "passive"))
@@
     (attr exclude_from_pos_files)
     (fp_text reference "LOGO1" (at 0 0) (layer "F.SilkS") hide
-      (effects (font (size 0.7 0.7) (thickness 0.127)))
+      (effects (font (size 0.8 0.8) (thickness 0.127)))
     )
     (fp_text value "Logo_Open_Hardware_Small" (at 0.75 0) (layer "F.Fab") hide
-      (effects (font (size 0.7 0.7) (thickness 0.127)))
+      (effects (font (size 0.8 0.8) (thickness 0.127)))
     )
     (fp_poly (pts
@@
     (attr smd)
     (fp_text reference "R1" (at 2.6 0 90) (layer "F.SilkS")
-      (effects (font (size 0.7 0.7) (thickness 0.127)))
+      (effects (font (size 0.8 0.8) (thickness 0.127)))
     )
     (fp_text value "10k" (at 0 1.43 90) (layer "F.Fab")
-      (effects (font (size 0.7 0.7) (thickness 0.127)))
+      (effects (font (size 0.8 0.8) (thickness 0.127)))
     )
     (fp_text user "${REFERENCE}" (at 0 0 90) (layer "F.Fab")
-      (effects (font (size 0.4 0.4) (thickness 0.06)))
+      (effects (font (size 0.8 0.8) (thickness 0.127)))
     )
     (fp_line (start -0.254724 -0.5225) (end 0.254724 -0.5225) (layer "F.SilkS") (width 0.12))
@@
       (net 1 "/SS443A/5V") (pintype "passive"))
     (pad "2" smd roundrect (at 0.9125 0 90) (size 0.975 0.95) (layers "F.Cu" "F.Paste" "F.Mask") (roundrect_rratio 0.25)
-      (net 10 "Net-(R1-Pad2)") (pintype "passive"))
+      (net 10 "Net-(Q1-Pad1)") (pintype "passive"))
     (model "${KICAD6_3DMODEL_DIR}/Resistor_SMD.3dshapes/R_0603_1608Metric.wrl"
       (offset (xyz 0 0 0))
@@
     (attr smd)
     (fp_text reference "C1" (at 2.7 0.1) (layer "F.SilkS")
-      (effects (font (size 0.7 0.7) (thickness 0.127)))
-    )
-    (fp_text value "0.1uF" (at 0 1.43) (layer "F.Fab")
-      (effects (font (size 0.7 0.7) (thickness 0.127)))
+      (effects (font (size 0.8 0.8) (thickness 0.127)))
+    )
+    (fp_text value "100nF" (at 0 1.43) (layer "F.Fab")
+      (effects (font (size 0.8 0.8) (thickness 0.127)))
     )
     (fp_text user "${REFERENCE}" (at 0 0) (layer "F.Fab")
-      (effects (font (size 0.4 0.4) (thickness 0.06)))
+      (effects (font (size 0.8 0.8) (thickness 0.127)))
     )
     (fp_line (start -0.146267 -0.51) (end 0.146267 -0.51) (layer "F.SilkS") (width 0.12))
@@
     (property "Sheetname" "SS443A")
     (fp_text reference "U1" (at -0.105 2.500007 90 unlocked) (layer "F.SilkS")
-      (effects (font (size 0.7 0.7) (thickness 0.127)) (justify left bottom))
+      (effects (font (size 0.8 0.8) (thickness 0.127)) (justify left bottom))
     )
     (fp_text value "SS443A" (at -1.968501 4.5085 180 unlocked) (layer "F.SilkS") hide
-      (effects (font (size 0.7 0.7) (thickness 0.127)) (justify left bottom))
+      (effects (font (size 0.8 0.8) (thickness 0.127)) (justify left bottom))
     )
     (fp_text user "${REFERENCE}" (at -0.459997 0.177841 180 unlocked) (layer "User.5")
-      (effects (font (size 0.5 0.5) (thickness 0.1)) (justify left bottom))
+      (effects (font (size 0.8 0.8) (thickness 0.127)) (justify left bottom))
     )
     (fp_line (start 1.3 -2.049998) (end 1.3 2.049998) (layer "F.SilkS") (width 0.2))
@@
       (net 2 "GND") (pinfunction "Ground(-)") (pintype "power_in") (solder_paste_margin -1000))
     (pad "3" thru_hole circle (at 0.164997 1.27 180) (size 1.2 1.2) (drill 0.7) (layers *.Cu *.Mask)
-      (net 10 "Net-(R1-Pad2)") (pinfunction "Output(O)") (pintype "passive") (solder_paste_margin -1000))
+      (net 10 "Net-(Q1-Pad1)") (pinfunction "Output(O)") (pintype "passive") (solder_paste_margin -1000))
     (model "${KIPRJMOD}/models/IC_Honeywell_SS443A_eec.STEP"
       (offset (xyz -0 -0 0))
@@
     (attr smd)
     (fp_text reference "R2" (at 0 1.4) (layer "F.SilkS")
-      (effects (font (size 0.7 0.7) (thickness 0.127)))
+      (effects (font (size 0.8 0.8) (thickness 0.127)))
     )
     (fp_text value "10k" (at 0 1.43) (layer "F.Fab")
-      (effects (font (size 0.7 0.7) (thickness 0.127)))
+      (effects (font (size 0.8 0.8) (thickness 0.127)))
     )
     (fp_text user "${REFERENCE}" (at 0 0) (layer "F.Fab")
-      (effects (font (size 0.4 0.4) (thickness 0.06)))
+      (effects (font (size 0.8 0.8) (thickness 0.127)))
     )
     (fp_line (start -0.254724 0.5225) (end 0.254724 0.5225) (layer "F.SilkS") (width 0.12))
